File: kicad/ravine.kicad_sch (KiCad schematic)
At the start: 77 parts, among them SW1 CherryMX, SW10 CherryMX, SW1001 CherryMX, SW1002 CherryMX, SW1003 CherryMX, SW1004 CherryMX, SW1005 CherryMX, SW1006 CherryMX, SW101 CherryMX, SW102 CherryMX, SW103 CherryMX, SW104 CherryMX, SW105 CherryMX, SW106 CherryMX, SW11 CherryMX, SW12 CherryMX, SW13 CherryMX, SW14 CherryMX, SW15 CherryMX, SW16 CherryMX, SW17 CherryMX, SW18 CherryMX, SW19 CherryMX, SW2 CherryMX, SW20 CherryMX, SW3 CherryMX, SW4 CherryMX, SW5 CherryMX, SW6 CherryMX, SW7 CherryMX, SW8 CherryMX, SW9 CherryMX

Commit message: evil things are happening
Parts:
- added D37, D38, D39, D40, D41, D42, D43, D44, D45, D46, D47, D48: D, symbol Device:D
- added SW27, SW28, SW29, SW30, SW31, SW32: CherryMX, symbol Switch:SW_Push
Connections:
- net P1: now also D37.1 (K), D38.2 (A), D39.2 (A)
- net P2: now also D40.2 (A), D41.1 (K), D42.2 (A)
- net P3: now also D43.2 (A), D44.2 (A), D45.1 (K)
- net interrupt: now also D46.1 (K), D47.1 (K), D48.1 (K)
- new net: D38.1 (K), SW27.1
- new net: D41.2 (A), D47.2 (A), SW27.2, SW32.2
- new net: D43.1 (K), SW31.1
- new net: D37.2 (A), D46.2 (A), SW29.2, SW31.2
- new net: D42.1 (K), SW30.1
- new net: D40.1 (K), SW29.1
- new net: D44.1 (K), SW32.1
- new net: D45.2 (A), D48.2 (A), SW28.2, SW30.2
- new net: D39.1 (K), SW28.1
Other:
- moved on the sheet: SW1, SW10, SW11, SW12, SW13, SW14, SW15, SW16, SW17, SW18, SW19, SW2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
